File: pcb/power/steve_power_distribution.kicad_pcb (KiCad board)
At the start: 2 copper layers, 50 x 50 mm, 19 parts, among them P1 BATT_1, P2 BATT_2, P3 BATT_3, P4 BATT_4, P5 MOTORS, P6 PI_5V, P7 AVR_5V, P8 AVR_INTERFACE, Q1 Q_NMOS_GDS, Q2 Q_NMOS_GDS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

Commit message: Finalized PCB design and generated gerbers for manufacture
Parts:
- added P11: MOUNT_HOLE, footprints:MOUNT_HOLE, F.Cu at (53.0, 147.0)
- added P12: MOUNT_HOLE, footprints:MOUNT_HOLE, F.Cu at (97.0, 147.0)
- added P13: MOUNT_HOLE, footprints:MOUNT_HOLE, F.Cu at (97.0, 103.0)
- added P14: MOUNT_HOLE, footprints:MOUNT_HOLE, F.Cu at (53.0, 103.0)
- added P5: BATT_AUX, Terminal_Blocks:TerminalBlock_Pheonix_PT-3.5mm_2pol, F.Cu at (61.5, 104.5)
- added P9: 5V_AUX, Terminal_Blocks:TerminalBlock_Pheonix_PT-3.5mm_2pol, F.Cu at (92.0, 104.5)
- P7: renamed from P6; value PI_5V -> 5V_PI
- P8: renamed from P7; value AVR_5V -> 5V_AVR
- moved P7 9.71 mm to (95.0, 114.5), turned to 90 degrees
- moved P6 6.32 mm to (55.0, 111.0), turned to 270 degrees
- moved P1 4.50 mm to (57.5, 145.0)
- moved P8 4.50 mm to (89.0, 145.0)
- moved P2 3.00 mm to (65.0, 145.0)
- moved P3 1.50 mm to (72.5, 145.0)
- moved U1 0.50 mm to (75.5, 129.5)
- renumbered P8 to P10, P5 to P6
Routing:
- net +5V: track 27.2 -> 0.00 mm
- net Net-(D2-Pad1): track 32.9 -> 22.5 mm
- net Net-(D1-Pad1): track 31.0 -> 27.3 mm
