File: pcb/power/steve_power_distribution.sch (KiCad schematic (older format))
At the start: 18 parts, among them P1 BATT_1, P2 BATT_2, P3 BATT_3, P4 BATT_4, P5 MOTORS, P6 PI_5V, P7 AVR_5V, Q1 Q_NMOS_GDS, Q2 Q_NMOS_GDS, U1 LM2596S_Carrier

Commit message: Semi finalized PCB layout
Parts:
- added P8: AVR_INTERFACE, Pin_Headers:Pin_Header_Straight_1x05, symbol CONN_01X05
Connections:
- net +5V: now also P8.1 (P1), P8.4 (P4)
- net EN_MOTORS: now also P8.2 (P2)
- net EN_PI: now also P8.5 (P5)
- net V_BATT: now also P8.3 (P3)
Changed lines of the file:
@@
 $EndComp
 $Comp
-L GND #PWR16
+L GND #PWR17
 U 1 1 57D57B43
 P 5850 2500
-F 0 "#PWR16" H 5850 2250 50  0001 C CNN
+F 0 "#PWR17" H 5850 2250 50  0001 C CNN
 F 1 "GND" H 5850 2350 50  0000 C CNN
 F 2 "" H 5850 2500 50  0000 C CNN
@@
 Connection ~ 5850 2450
 $Comp
-L GND #PWR20
+L GND #PWR21
 U 1 1 57D57D83
 P 5850 4850
-F 0 "#PWR20" H 5850 4600 50  0001 C CNN
+F 0 "#PWR21" H 5850 4600 50  0001 C CNN
 F 1 "GND" H 5850 4700 50  0000 C CNN
 F 2 "" H 5850 4850 50  0000 C CNN
@@
 $EndComp
 $Comp
-L GND #PWR18
+L GND #PWR19
 U 1 1 57D58D3D
 P 5850 4000
-F 0 "#PWR18" H 5850 3750 50  0001 C CNN
+F 0 "#PWR19" H 5850 3750 50  0001 C CNN
 F 1 "GND" H 5850 3850 50  0000 C CNN
 F 2 "" H 5850 4000 50  0000 C CNN
@@
 $EndComp
 $Comp
-L +5V #PWR19
+L +5V #PWR20
 U 1 1 57D5925B
 P 5850 4750
-F 0 "#PWR19" H 5850 4600 50  0001 C CNN
+F 0 "#PWR20" H 5850 4600 50  0001 C CNN
 F 1 "+5V" H 5850 4890 50  0000 C CNN
 F 2 "" H 5850 4750 50  0000 C CNN
@@
 $EndComp
 $Comp
-L +5V #PWR17
+L +5V #PWR18
 U 1 1 57D59930
 P 5850 3050
-F 0 "#PWR17" H 5850 2900 50  0001 C CNN
+F 0 "#PWR18" H 5850 2900 50  0001 C CNN
 F 1 "+5V" H 5850 3190 50  0000 C CNN
 F 2 "" H 5850 3050 50  0000 C CNN
@@
 $EndComp
 $Comp
-L +BATT #PWR15
+L +BATT #PWR16
 U 1 1 57D5A008
 P 5850 1550
-F 0 "#PWR15" H 5850 1400 50  0001 C CNN
+F 0 "#PWR16" H 5850 1400 50  0001 C CNN
 F 1 "+BATT" H 5850 1690 50  0000 C CNN
 F 2 "" H 5850 1550 50  0000 C CNN
@@
 $EndComp
 Wire Wire Line
-	5850 1850 5850 1650
+	5850 1650 5850 1850
 Wire Wire Line
 	5450 2150 5450 2050
@@
 Connection ~ 5450 3550
 Wire Wire Line
-	5850 3350 5850 3150
+	5850 3150 5850 3350
 Text Label 3800 2850 0    60   ~ 0
 V_BATT
@@
 	6600 1800 5850 1800
 Connection ~ 5850 1800
+$Comp
+L CONN_01X05 P8
+U 1 1 57D5EFD8
+P 6050 5650
+F 0 "P8" H 6050 5950 50  0000 C CNN
+F 1 "AVR_INTERFACE" V 6150 5650 50  0000 C CNN
+F 2 "Pin_Headers:Pin_Header_Straight_1x05" H 6050 5650 50  0001 C CNN
+F 3 "" H 6050 5650 50  0000 C CNN
+	1    6050 5650
+	1    0    0    -1
+$EndComp
+$Comp
+L +5V #PWR15
+U 1 1 57D5F84A
+P 5250 5350
+F 0 "#PWR15" H 5250 5200 50  0001 C CNN
+F 1 "+5V" H 5250 5490 50  0000 C CNN
+F 2 "" H 5250 5350 50  0000 C CNN
+F 3 "" H 5250 5350 50  0000 C CNN
+	1    5250 5350
+	1    0    0    -1
+$EndComp
+Text Label 5850 5650 2    60   ~ 0
+V_BATT
+Text Label 5850 5550 2    60   ~ 0
+EN_MOTORS
+Text Label 5850 5850 2    60   ~ 0
+EN_PI
+Wire Wire Line
+	5250 5350 5250 5750
+Wire Wire Line
+	5250 5450 5850 5450
+Connection ~ 5250 5450
+Wire Wire Line
+	5250 5750 5850 5750
 $EndSCHEMATC

Commit message: Finalized PCB design and generated gerbers for manufacture
Parts:
- added P11, P12, P13, P14: MOUNT_HOLE, footprints:MOUNT_HOLE, symbol CONN_01X01
- added P5: BATT_AUX, Terminal_Blocks:TerminalBlock_Pheonix_PT-3.5mm_2pol, symbol CONN_01X02
- added P9: 5V_AUX, Terminal_Blocks:TerminalBlock_Pheonix_PT-3.5mm_2pol, symbol CONN_01X02
- P7: renamed from P6; value PI_5V -> 5V_PI
- P8: renamed from P7; value AVR_5V -> 5V_AVR
- renumbered P8 to P10, P5 to P6
Connections:
- net +5V: now also P9.2 (P2)
- net +BATT: now also P5.2 (P2)
- net GND: now also P5.1 (P1), P9.1 (P1)
Other:
- moved on the sheet: P10, P8
Changed lines of the file:
@@
 $EndComp
 $Comp
-L CONN_01X02 P5
+L CONN_01X02 P6
 U 1 1 57D5611B
 P 6050 1600
-F 0 "P5" H 6050 1750 50  0000 C CNN
+F 0 "P6" H 6050 1750 50  0000 C CNN
 F 1 "MOTORS" V 6150 1600 50  0000 C CNN
 F 2 "Terminal_Blocks:TerminalBlock_Pheonix_PT-3.5mm_2pol" H 6050 1600 50  0001 C CNN
@@
 $EndComp
 $Comp
-L CONN_01X02 P6
+L CONN_01X02 P7
 U 1 1 57D563BC
 P 6050 3100
-F 0 "P6" H 6050 3250 50  0000 C CNN
-F 1 "PI_5V" V 6150 3100 50  0000 C CNN
+F 0 "P7" H 6050 3250 50  0000 C CNN
+F 1 "5V_PI" V 6150 3100 50  0000 C CNN
 F 2 "Terminal_Blocks:TerminalBlock_Pheonix_PT-3.5mm_2pol" H 6050 3100 50  0001 C CNN
 F 3 "" H 6050 3100 50  0000 C CNN
@@
 $EndComp
 $Comp
-L CONN_01X02 P7
+L CONN_01X02 P8
 U 1 1 57D564C7
-P 6050 4800
-F 0 "P7" H 6050 4950 50  0000 C CNN
-F 1 "AVR_5V" V 6150 4800 50  0000 C CNN
-F 2 "Terminal_Blocks:TerminalBlock_Pheonix_PT-3.5mm_2pol" H 6050 4800 50  0001 C CNN
-F 3 "" H 6050 4800 50  0000 C CNN
-	1    6050 4800
+P 6050 4550
+F 0 "P8" H 6050 4700 50  0000 C CNN
+F 1 "5V_AVR" V 6150 4550 50  0000 C CNN
+F 2 "Terminal_Blocks:TerminalBlock_Pheonix_PT-3.5mm_2pol" H 6050 4550 50  0001 C CNN
+F 3 "" H 6050 4550 50  0000 C CNN
+	1    6050 4550
 	1    0    0    1
 $EndComp
@@
 $EndComp
 $Comp
-L GND #PWR12
+L GND #PWR14
 U 1 1 57D577A5
 P 3450 3200
-F 0 "#PWR12" H 3450 2950 50  0001 C CNN
+F 0 "#PWR14" H 3450 2950 50  0001 C CNN
 F 1 "GND" H 3450 3050 50  0000 C CNN
 F 2 "" H 3450 3200 50  0000 C CNN
@@
 $EndComp
 $Comp
-L GND #PWR17
+L GND #PWR19
 U 1 1 57D57B43
 P 5850 2500
-F 0 "#PWR17" H 5850 2250 50  0001 C CNN
+F 0 "#PWR19" H 5850 2250 50  0001 C CNN
 F 1 "GND" H 5850 2350 50  0000 C CNN
 F 2 "" H 5850 2500 50  0000 C CNN
@@
 Connection ~ 5850 2450
 $Comp
-L GND #PWR21
+L GND #PWR23
 U 1 1 57D57D83
-P 5850 4850
-F 0 "#PWR21" H 5850 4600 50  0001 C CNN
-F 1 "GND" H 5850 4700 50  0000 C CNN
-F 2 "" H 5850 4850 50  0000 C CNN
-F 3 "" H 5850 4850 50  0000 C CNN
-	1    5850 4850
-	1    0    0    -1
-$EndComp
-$Comp
-L GND #PWR10
+P 5850 4600
+F 0 "#PWR23" H 5850 4350 50  0001 C CNN
+F 1 "GND" H 5850 4450 50  0000 C CNN
+F 2 "" H 5850 4600 50  0000 C CNN
+F 3 "" H 5850 4600 50  0000 C CNN
+	1    5850 4600
+	1    0    0    -1
+$EndComp
+$Comp
+L GND #PWR12
 U 1 1 57D58365
 P 2950 5450
-F 0 "#PWR10" H 2950 5200 50  0001 C CNN
+F 0 "#PWR12" H 2950 5200 50  0001 C CNN
 F 1 "GND" H 2950 5300 50  0000 C CNN
 F 2 "" H 2950 5450 50  0000 C CNN
@@
 $EndComp
 $Comp
-L GND #PWR14
+L GND #PWR16
 U 1 1 57D584C2
 P 4150 5450
-F 0 "#PWR14" H 4150 5200 50  0001 C CNN
+F 0 "#PWR16" H 4150 5200 50  0001 C CNN
 F 1 "GND" H 4150 5300 50  0000 C CNN
 F 2 "" H 4150 5450 50  0000 C CNN
@@
 $EndComp
 $Comp
-L GND #PWR19
+L GND #PWR21
 U 1 1 57D58D3D
 P 5850 4000
-F 0 "#PWR19" H 5850 3750 50  0001 C CNN
+F 0 "#PWR21" H 5850 3750 50  0001 C CNN
 F 1 "GND" H 5850 3850 50  0000 C CNN
 F 2 "" H 5850 4000 50  0000 C CNN
@@
 Connection ~ 5850 3950
 $Comp
-L +5V #PWR13
+L +5V #PWR15
 U 1 1 57D59219
 P 4150 4850
-F 0 "#PWR13" H 4150 4700 50  0001 C CNN
+F 0 "#PWR15" H 4150 4700 50  0001 C CNN
 F 1 "+5V" H 4150 4990 50  0000 C CNN
 F 2 "" H 4150 4850 50  0000 C CNN
@@
 $EndComp
 $Comp
+L +5V #PWR22
+U 1 1 57D5925B
+P 5850 4500
+F 0 "#PWR22" H 5850 4350 50  0001 C CNN
+F 1 "+5V" H 5850 4640 50  0000 C CNN
+F 2 "" H 5850 4500 50  0000 C CNN
+F 3 "" H 5850 4500 50  0000 C CNN
+	1    5850 4500
+	1    0    0    -1
+$EndComp
+$Comp
 L +5V #PWR20
-U 1 1 57D5925B
-P 5850 4750
-F 0 "#PWR20" H 5850 4600 50  0001 C CNN
-F 1 "+5V" H 5850 4890 50  0000 C CNN
-F 2 "" H 5850 4750 50  0000 C CNN
-F 3 "" H 5850 4750 50  0000 C CNN
-	1    5850 4750
-	1    0    0    -1
-$EndComp
-$Comp
-L +5V #PWR18
 U 1 1 57D59930
 P 5850 3050
-F 0 "#PWR18" H 5850 2900 50  0001 C CNN
+F 0 "#PWR20" H 5850 2900 50  0001 C CNN
 F 1 "+5V" H 5850 3190 50  0000 C CNN
 F 2 "" H 5850 3050 50  0000 C CNN
@@
 $EndComp
 $Comp
-L +BATT #PWR9
+L +BATT #PWR11
 U 1 1 57D59C72
 P 2950 4850
-F 0 "#PWR9" H 2950 4700 50  0001 C CNN
+F 0 "#PWR11" H 2950 4700 50  0001 C CNN
 F 1 "+BATT" H 2950 4990 50  0000 C CNN
 F 2 "" H 2950 4850 50  0000 C CNN
@@
 $EndComp
 $Comp
-L +BATT #PWR11
+L +BATT #PWR13
 U 1 1 57D59E9D
 P 3450 2500
-F 0 "#PWR11" H 3450 2350 50  0001 C CNN
+F 0 "#PWR13" H 3450 2350 50  0001 C CNN
 F 1 "+BATT" H 3450 2640 50  0000 C CNN
 F 2 "" H 3450 2500 50  0000 C CNN
@@
 $EndComp
 $Comp
-L +BATT #PWR16
+L +BATT #PWR18
 U 1 1 57D5A008
 P 5850 1550
-F 0 "#PWR16" H 5850 1400 50  0001 C CNN
+F 0 "#PWR18" H 5850 1400 50  0001 C CNN
 F 1 "+BATT" H 5850 1690 50  0000 C CNN
 F 2 "" H 5850 1550 50  0000 C CNN
@@
 Connection ~ 5850 1800
 $Comp
-L CONN_01X05 P8
+L CONN_01X05 P10
 U 1 1 57D5EFD8
-P 6050 5650
-F 0 "P8" H 6050 5950 50  0000 C CNN
-F 1 "AVR_INTERFACE" V 6150 5650 50  0000 C CNN
-F 2 "Pin_Headers:Pin_Header_Straight_1x05" H 6050 5650 50  0001 C CNN
-F 3 "" H 6050 5650 50  0000 C CNN
-	1    6050 5650
-	1    0    0    -1
-$EndComp
-$Comp
-L +5V #PWR15
+P 6050 6000
+F 0 "P10" H 6050 6300 50  0000 C CNN
+F 1 "AVR_INTERFACE" V 6150 6000 50  0000 C CNN
+F 2 "Pin_Headers:Pin_Header_Straight_1x05" H 6050 6000 50  0001 C CNN
+F 3 "" H 6050 6000 50  0000 C CNN
+	1    6050 6000
+	1    0    0    -1
+$EndComp
+$Comp
+L +5V #PWR17
 U 1 1 57D5F84A
-P 5250 5350
-F 0 "#PWR15" H 5250 5200 50  0001 C CNN
-F 1 "+5V" H 5250 5490 50  0000 C CNN
-F 2 "" H 5250 5350 50  0000 C CNN
-F 3 "" H 5250 5350 50  0000 C CNN
-	1    5250 5350
-	1    0    0    -1
-$EndComp
-Text Label 5850 5650 2    60   ~ 0
+P 5250 5700
+F 0 "#PWR17" H 5250 5550 50  0001 C CNN
+F 1 "+5V" H 5250 5840 50  0000 C CNN
+F 2 "" H 5250 5700 50  0000 C CNN
+F 3 "" H 5250 5700 50  0000 C CNN
+	1    5250 5700
+	1    0    0    -1
+$EndComp
+Text Label 5850 6000 2    60   ~ 0
 V_BATT
-Text Label 5850 5550 2    60   ~ 0
+Text Label 5850 5900 2    60   ~ 0
 EN_MOTORS
-Text Label 5850 5850 2    60   ~ 0
+Text Label 5850 6200 2    60   ~ 0
 EN_PI
 Wire Wire Line
-	5250 5350 5250 5750
-Wire Wire Line
-	5250 5450 5850 5450
-Connection ~ 5250 5450
-Wire Wire Line
-	5250 5750 5850 5750
+	5250 5700 5250 6100
+Wire Wire Line
+	5250 5800 5850 5800
+Connection ~ 5250 5800
+Wire Wire Line
+	5250 6100 5850 6100
+$Comp
+L CONN_01X02 P9
+U 1 1 57D863AB
+P 6050 5200
+F 0 "P9" H 6050 5350 50  0000 C CNN
+F 1 "5V_AUX" V 6150 5200 50  0000 C CNN
+F 2 "Terminal_Blocks:TerminalBlock_Pheonix_PT-3.5mm_2pol" H 6050 5200 50  0001 C CNN
+F 3 "" H 6050 5200 50  0000 C CNN
+	1    6050 5200
+	1    0    0    1
+$EndComp
+$Comp
+L GND #PWR25
+U 1 1 57D863B1
+P 5850 5250
+F 0 "#PWR25" H 5850 5000 50  0001 C CNN
+F 1 "GND" H 5850 5100 50  0000 C CNN
+F 2 "" H 5850 5250 50  0000 C CNN
+F 3 "" H 5850 5250 50  0000 C CNN
+	1    5850 5250
+	1    0    0    -1
+$EndComp
+$Comp
+L +5V #PWR24
+U 1 1 57D863B7
+P 5850 5150
+F 0 "#PWR24" H 5850 5000 50  0001 C CNN
+F 1 "+5V" H 5850 5290 50  0000 C CNN
+F 2 "" H 5850 5150 50  0000 C CNN
+F 3 "" H 5850 5150 50  0000 C CNN
+	1    5850 5150
+	1    0    0    -1
+$EndComp
+$Comp
+L CONN_01X01 P11
+U 1 1 57D87118
+P 9650 1250
+F 0 "P11" H 9650 1350 50  0000 C CNN
+F 1 "MOUNT_HOLE" V 9750 1250 50  0000 C CNN
+F 2 "footprints:MOUNT_HOLE" H 9650 1250 50  0001 C CNN
+F 3 "" H 9650 1250 50  0000 C CNN
+	1    9650 1250
+	1    0    0    -1
+$EndComp
+$Comp
+L CONN_01X01 P12
+U 1 1 57D871A3
+P 9650 1800
+F 0 "P12" H 9650 1900 50  0000 C CNN
+F 1 "MOUNT_HOLE" V 9750 1800 50  0000 C CNN
+F 2 "footprints:MOUNT_HOLE" H 9650 1800 50  0001 C CNN
+F 3 "" H 9650 1800 50  0000 C CNN
+	1    9650 1800
+	1    0    0    -1
+$EndComp
+$Comp
+L CONN_01X01 P13
+U 1 1 57D8720D
+P 9650 2350
+F 0 "P13" H 9650 2450 50  0000 C CNN
+F 1 "MOUNT_HOLE" V 9750 2350 50  0000 C CNN
+F 2 "footprints:MOUNT_HOLE" H 9650 2350 50  0001 C CNN
+F 3 "" H 9650 2350 50  0000 C CNN
+	1    9650 2350
+	1    0    0    -1
+$EndComp
+$Comp
+L CONN_01X01 P14
+U 1 1 57D87274
+P 9650 2900
+F 0 "P14" H 9650 3000 50  0000 C CNN
+F 1 "MOUNT_HOLE" V 9750 2900 50  0000 C CNN
+F 2 "footprints:MOUNT_HOLE" H 9650 2900 50  0001 C CNN
+F 3 "" H 9650 2900 50  0000 C CNN
+	1    9650 2900
+	1    0    0    -1
+$EndComp
+$Comp
+L CONN_01X02 P5
+U 1 1 57D88027
+P 1200 4750
+F 0 "P5" H 1200 4900 50  0000 C CNN
+F 1 "BATT_AUX" V 1300 4750 50  0000 C CNN
+F 2 "Terminal_Blocks:TerminalBlock_Pheonix_PT-3.5mm_2pol" H 1200 4750 50  0001 C CNN
+F 3 "" H 1200 4750 50  0000 C CNN
+	1    1200 4750
+	-1   0    0    1
+$EndComp
+$Comp
+L GND #PWR10
+U 1 1 57D8802D
+P 1400 4800
+F 0 "#PWR10" H 1400 4550 50  0001 C CNN
+F 1 "GND" H 1400 4650 50  0000 C CNN
+F 2 "" H 1400 4800 50  0000 C CNN
+F 3 "" H 1400 4800 50  0000 C CNN
+	1    1400 4800
+	1    0    0    -1
+$EndComp
+$Comp
+L +BATT #PWR9
+U 1 1 57D88033
+P 1400 4700
+F 0 "#PWR9" H 1400 4550 50  0001 C CNN
+F 1 "+BATT" H 1400 4840 50  0000 C CNN
+F 2 "" H 1400 4700 50  0000 C CNN
+F 3 "" H 1400 4700 50  0000 C CNN
+	1    1400 4700
+	1    0    0    -1
+$EndComp
 $EndSCHEMATC
